File: kicad/ESP32-Automatic-Optical-Audio-Switch.kicad_sch (KiCad schematic)
At the start: 31 parts, among them IC1 74LVC1G157GW,125, J1 FC684208R, J2 FC684208R, U1 74AHC1G4212, U2 74AHC1G4212, U3 ESP32-S3-ZERO, U4 FCR684208T, U5 AP2127K-3.3

Commit message: Add system diagram and update PCB for ESP32 switch
Added a Draw.io system diagram for the ESP32 Optical Audio Switch. Updated the KiCad PCB and schematic files to reference the correct sheet file and replaced a capacitor footprint with the ESP32-C3-ZERO module footprint. Also updated .gitignore to exclude temporary Draw.io files.
Parts:
- removed U3: ESP32-S3-ZERO, footprints:MODULE_ESP32-S3-ZERO, symbol ESP32-S3-ZERO:ESP32-S3-ZERO
- added U3: ESP32-C3-ZERO, footprints:MODULE_ESP32-C3-ZERO, symbol ESP32-S3-ZERO:ESP32-C3-ZERO
- IC1: footprint footprints:SOP65P210X110-6N -> SOP65P210X110-6N
Connections:
- net CH_A_DIV: now also U3.1 (GP1)
- net CH_B_DIV: now also U3.2 (GP2)
- net GND: now also U3.GND
- net SW_CH_B: now also U3.5 (GP5)
- net at L1.1: now also U3.5V
